Commit message: some parameter tuning

File: fav_sim/models/bluerov/urdf/bluerov_params.xacro (robot description, xacro)
@@ -2,7 +2,7 @@
 <robot xmlns:xacro="http://www.ros.org/wiki/xacro">
     <xacro:property name="base_mass" value="11.0" />
-    <xacro:property name="ixx" value="0.05" />
-    <xacro:property name="iyy" value="0.05" />
-    <xacro:property name="izz" value="0.05" />
+    <xacro:property name="ixx" value="0.005" />
+    <xacro:property name="iyy" value="0.005" />
+    <xacro:property name="izz" value="0.2" />
     <xacro:property name="added_mass_linear" value="0 0 0" />
     <xacro:property name="added_mass_angular" value="0 0 0" />

File: fav_sim/models/thruster/urdf/thruster_macro.xacro (robot description, xacro)
@@ -26,5 +26,5 @@
                 <torque_coeff>${torque_constant}</torque_coeff>
                 <rpm_scaler>${rpm_scaler}</rpm_scaler>
-                <max_rpm>${max_rpm}</max_rpm>
+                <maximum_rpm>${maximum_rpm}</maximum_rpm>
                 <thruster_number>${number}</thruster_number>
                 <turning_direction>${turning_direction}</turning_direction>

File: fav_sim/models/thruster/urdf/thruster_params.xacro (robot description, xacro)
@@ -5,9 +5,9 @@
     <xacro:property name="thruster_iyy" value="1e-6" />
     <xacro:property name="thruster_izz" value="1e-6" />
-    <xacro:property name="thrust_linear_coeff" value="15.89e-5" />
-    <xacro:property name="thrust_quadratic_coeff" value="23.2e-5" />
+    <xacro:property name="thrust_linear_coeff" value="-0.053" />
+    <xacro:property name="thrust_quadratic_coeff" value="0.016" />
     <xacro:property name="torque_constant" value="1e-2" />
     <xacro:property name="rpm_scaler" value="1" />
-    <xacro:property name="max_rpm" value="800" />
+    <xacro:property name="maximum_rpm" value="1280" />
     <xacro:property name="timeconstant_up" value="0.05" />
     <xacro:property name="timeconstant_down" value="0.05" />
