Commit message: esc_commander added

File: fav_sim/models/bluerov/urdf/bluerov.xacro (robot description, xacro)
@@ -4,15 +4,12 @@
     <xacro:include filename="$(find fav_sim)/models/thruster/urdf/thruster_macro.xacro" />
     <xacro:property name="thruster_xy" value="${thruster_r / 2**0.5}" />
-    <gazebo>
-        <static>false</static>
-    </gazebo>
     <link name="base_link">
-        <inertial>
+        <inertial name="base_link_inertial">
             <mass value="${base_mass}" />
             <inertia ixx="${ixx}" ixy="0.0" ixz="0.0" iyy="${iyy}" iyz="0.0" izz="${izz}" />
         </inertial>
-        <visual>
+        <visual name="base_link_visual">
             <geometry>
-                <mesh filename="$(find fav_sim)/models/bluerov/meshes/bluerov.dae" />
+                <mesh filename="file://$(find fav_sim)/models/bluerov/meshes/bluerov.dae" />
             </geometry>
         </visual>
@@ -29,4 +26,17 @@
             <damping_angular>${damping_angular}</damping_angular>
         </plugin>
+        <plugin name="joint_state" filename="libgazebo_ros_joint_state_publisher.so">
+            <robotNamespace />
+            <jointName>front_starboard_horizontal_thruster_propeller_joint,
+                front_port_horizontal_thruster_propeller_joint,
+                rear_starboard_horizontal_thruster_propeller_joint,
+                rear_port_horizontal_thruster_propeller_joint,
+                front_starboard_vertical_thruster_propeller_joint,
+                front_port_vertical_thruster_propeller_joint,
+                rear_starboard_vertical_thruster_propeller_joint,
+                rear_port_vertical_thruster_propeller_joint
+            </jointName>
+            <updateRate>50.0</updateRate>
+        </plugin>
     </gazebo>
     <xacro:thruster parent="base_link" suffix="front_starboard_horizontal" xyz="0.14 -0.10 0" rpy="0 0 ${radians(45)}" turning_direction="cw" propeller_direction="cw" color="red" number="0" />

File: fav_sim/models/thruster/urdf/thruster_macro.xacro (robot description, xacro)
@@ -7,16 +7,16 @@
         <link name="${propeller_link}">
             <origin xyz="0 0 0" rpy="0 0 0" />
-            <inertial>
+            <inertial name="${propeller_link}_inertial">
                 <mass value="${thruster_mass}" />
                 <inertia ixx="${thruster_ixx}" ixy="0.0" ixz="0.0" iyy="${thruster_iyy}" iyz="0.0" izz="${thruster_izz}" />
             </inertial>
-            <visual>
+            <visual name="${propeller_link}_visual">
                 <geometry>
-                    <mesh filename="$(find fav_sim)/models/thruster/meshes/propeller.dae" />
+                    <mesh filename="file://$(find fav_sim)/models/thruster/meshes/propeller.dae" />
                 </geometry>
             </visual>
         </link>
         <gazebo>
-            <plugin name="thruster" filename="libthruster.so">
+            <plugin name="${suffix}_thruster" filename="libthruster.so">
                 <link>${propeller_link}</link>
                 <joint>${propeller_joint}</joint>

Commit message: added barometer

File: fav_sim/models/bluerov/urdf/bluerov.xacro (robot description, xacro)
@@ -26,4 +26,9 @@
             <damping_angular>${damping_angular}</damping_angular>
         </plugin>
+        <plugin name="barometer" filename="libbarometer.so">
+            <link>base_link</link>
+            <position>${barometer_position}</position>
+            <noise>${barometer_noise}</noise>
+        </plugin>
         <plugin name="joint_state" filename="libgazebo_ros_joint_state_publisher.so">
             <robotNamespace />

File: fav_sim/models/bluerov/urdf/bluerov_params.xacro (robot description, xacro)
@@ -11,3 +11,5 @@
     <xacro:property name="buoyancy_compensation" value="1.001" />
     <xacro:property name="buoyancy_origin" value="0 0 0.005" />
+    <xacro:property name="barometer_position" value="-0.15 0 -0.05" />
+    <xacro:property name="barometer_noise" value="100.0" />
 </robot>

Commit message: imu added

File: fav_sim/models/bluerov/urdf/bluerov.xacro (robot description, xacro)
@@ -53,5 +53,38 @@
             <xyzOffsets>0 0 0</xyzOffsets>
             <rpyOffsets>0 0 0</rpyOffsets>
-          </plugin>
+        </plugin>
+    </gazebo>
+    <gazebo reference="imu_link">
+        <sensor name="imu_sensor" type="imu">
+            <always_on>true</always_on>
+            <update_rate>100</update_rate>
+            <visualize>true</visualize>
+            <topic>__default_topic__</topic>
+            <plugin filename="libgazebo_ros_imu_sensor.so" name="imu_plugin">
+                <topicName>imu/data</topicName>
+                <bodyName>imu_link</bodyName>
+                <updateRateHZ>50.0</updateRateHZ>
+                <gaussianNoise>0.0</gaussianNoise>
+                <xyzOffset>0 0 0</xyzOffset>
+                <rpyOffset>0 0 0</rpyOffset>
+                <frameName>imu</frameName>
+                <initialOrientationAsReference>false</initialOrientationAsReference>
+            </plugin>
+            <pose>0 0 0 0 0 0</pose>
+        </sensor>
+    </gazebo>
+    <link name="imu_link">
+        <inertial name="base_link_inertial">
+            <mass value="1e-5" />
+            <inertia ixx="1e-6" ixy="0" ixz="0" iyy="1e-6" iyz="0.0" izz="1e-6" />
+        </inertial>
+    </link>
+    <joint name="imu_joint" type="fixed">
+        <origin xyz="${imu_position}" rpy="${imu_orientation}" />
+        <parent link="base_link" />
+        <child link="imu_link" />
+    </joint>
+    <gazebo reference="imu_joint">
+        <preserveFixedJoint>true</preserveFixedJoint>
     </gazebo>
     <xacro:thruster parent="base_link" suffix="front_starboard_horizontal" xyz="0.14 -0.10 0" rpy="0 0 ${radians(45)}" turning_direction="cw" propeller_direction="cw" color="red" number="0" />

File: fav_sim/models/bluerov/urdf/bluerov_params.xacro (robot description, xacro)
@@ -13,3 +13,7 @@
     <xacro:property name="barometer_position" value="-0.15 0 -0.05" />
     <xacro:property name="barometer_noise" value="100.0" />
+    <!-- relative to the BlueROV's body-frame -->
+    <xacro:property name="imu_position" value="0.15 0 0.05" />
+    <xacro:property name="imu_orientation" value="${radians(0)} ${radians(0)} ${radians(0)}"/>
+    <xacro:property name="imu_noise" value="0.0003"/>
 </robot>

Commit message: added range_sensor for assignment 2

File: fav_sim/models/bluerov/urdf/bluerov.xacro (robot description, xacro)
@@ -3,4 +3,5 @@
     <xacro:include filename="$(find fav_sim)/models/bluerov/urdf/bluerov_params.xacro" />
     <xacro:include filename="$(find fav_sim)/models/thruster/urdf/thruster_macro.xacro" />
+    <xacro:include filename="$(find fav_sim)/models/range_sensor/urdf/range_sensor_macro.xacro" />
     <xacro:property name="thruster_xy" value="${thruster_r / 2**0.5}" />
     <link name="base_link">
@@ -96,4 +97,4 @@
     <xacro:thruster parent="base_link" suffix="rear_starboard_vertical" xyz="-0.12 -0.22 0.06" rpy="0 ${radians(-90)} 0" turning_direction="ccw" propeller_direction="cw" color="grey" number="6" />
     <xacro:thruster parent="base_link" suffix="rear_port_vertical" xyz="-0.12 0.22 0.06" rpy="0 ${radians(-90)} 0" turning_direction="cw" propeller_direction="cw" color="grey" number="7" />
-    <!-- <xacro:camera_macro parent="base_link" prefix="vertical_camera" xyz="${camera_position}" rpy="0 ${radians(90)} 0" /> -->
+    <xacro:range_sensor parent="base_link" prefix="range_sensor" xyz="${range_sensor_position}" rpy="${range_sensor_orientation}" />
 </robot>

File: fav_sim/models/bluerov/urdf/bluerov_params.xacro (robot description, xacro)
@@ -17,3 +17,5 @@
     <xacro:property name="imu_orientation" value="${radians(0)} ${radians(0)} ${radians(0)}"/>
     <xacro:property name="imu_noise" value="0.0003"/>
+    <xacro:property name="range_sensor_position" value="0.2 0 0.1" />
+    <xacro:property name="range_sensor_orientation" value="${radians(0)} ${radians(0)} ${radians(0)}" />
 </robot>

Commit message: added optional cameras to robot description

File: fav_sim/models/bluerov/urdf/bluerov.xacro (robot description, xacro)
@@ -4,4 +4,5 @@
     <xacro:include filename="$(find fav_sim)/models/thruster/urdf/thruster_macro.xacro" />
     <xacro:include filename="$(find fav_sim)/models/range_sensor/urdf/range_sensor_macro.xacro" />
+    <xacro:include filename="$(find fav_sim)/models/camera/urdf/camera_macro.xacro" />
     <xacro:property name="thruster_xy" value="${thruster_r / 2**0.5}" />
     <link name="base_link">
@@ -89,4 +90,10 @@
         <preserveFixedJoint>true</preserveFixedJoint>
     </gazebo>
+    <xacro:if value="$(arg use_vertical_camera)">
+        <xacro:camera parent="base_link" prefix="vertical_camera" xyz="${vertical_camera_position}" rpy="${vertical_camera_orientation}" />
+    </xacro:if>
+    <xacro:if value="$(arg use_front_camera)">
+        <xacro:camera parent="base_link" prefix="front_camera" xyz="${front_camera_position}" rpy="${front_camera_orientation}" />
+    </xacro:if>
     <xacro:thruster parent="base_link" suffix="front_starboard_horizontal" xyz="0.14 -0.10 0" rpy="0 0 ${radians(45)}" turning_direction="cw" propeller_direction="cw" color="red" number="0" />
     <xacro:thruster parent="base_link" suffix="front_port_horizontal" xyz="0.14 0.10 0" rpy="0 0 ${radians(-45)}" turning_direction="cw" propeller_direction="cw" color="green" number="1" />

File: fav_sim/models/bluerov/urdf/bluerov_params.xacro (robot description, xacro)
@@ -19,3 +19,10 @@
     <xacro:property name="range_sensor_position" value="0.2 0 0.1" />
     <xacro:property name="range_sensor_orientation" value="${radians(0)} ${radians(0)} ${radians(0)}" />
+    <xacro:arg name="use_vertical_camera" default="false" />
+    <xacro:property name="vertical_camera_position" value="0.15 0 -0.08" />
+    <xacro:property name="vertical_camera_orientation" value="0 ${radians(90)} 0" />
+    <xacro:arg name="use_front_camera" default="false" />
+    <!-- probably we want this to be the same as the range sensor position -->
+    <xacro:property name="front_camera_position" value="0.2 0 0.1" />
+    <xacro:property name="front_camera_orientation" value="0 0 0" />
 </robot>
