Commit message: added more parameters

File: fav_sim/models/range_sensor/urdf/range_sensor_macro.xacro (robot description, xacro)
@@ -24,6 +24,6 @@
                 <topic>ranges</topic>
                 <range_noise_std>${noise_stddev}</range_noise_std>
-                <max_fov_angle>100</max_fov_angle>
-                <max_viewing_angle>140</max_viewing_angle>
+                <max_fov_angle>${max_fov_angle}</max_fov_angle>
+                <max_viewing_angle>${max_viewing_angle}</max_viewing_angle>
                 <drop_probability>${drop_probability}</drop_probability>
                 <max_detection_distance>${max_detection_distance}</max_detection_distance>

File: fav_sim/models/range_sensor/urdf/range_sensor_params.xacro (robot description, xacro)
@@ -7,3 +7,10 @@
     <!-- scaling coefficient of a measurement beeing dropped due to the distance -->
     <xacro:property name="drop_probability_exponent" value="2.0" />
+    <!-- angle limit between x-axis of the robot and the normal axis of the
+        detected range target. For larger angles, no range measurement will
+        be generated -->
+    <xacro:property name="max_viewing_angle" value="140.0" />
+    <!-- field of view angle of the range sensor. Tags outside this cone won't
+        be detected. -->
+    <xacro:property name="max_fov_angle" value="90.0" />
 </robot>
